File: Carte_Base_roulante_2024.kicad_sch (KiCad schematic)
At the start: 64 parts, among them J11 ENC1, J16 ALIM, J4 ENC2, J5 ENC3, Q2 IRF7424, U1 STM32G484RETx

Commit message: compact : alim, encodeur, imu
Parts:
- C1, C10, C11, C12, C13, C14, C15, C16, C17, C18, C19, C20, C21, C22, C3, C5, C7, C8, C9: footprint Capacitor_SMD:C_0805_2012Metric -> Capacitor_SMD:C_0603_1608Metric
- C23, C24: footprint Capacitor_SMD:C_1206_3216Metric -> Capacitor_SMD:C_0603_1608Metric
Changed lines of the file:
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@@
       (effects (font (size 1.27 1.27)) (justify left))
     )
-    (property "Footprint" "Capacitor_SMD:C_0805_2012Metric" (at 157.1752 40.64 0)
+    (property "Footprint" "Capacitor_SMD:C_0603_1608Metric" (at 157.1752 40.64 0)
       (effects (font (size 1.27 1.27)) hide)
     )
@@
       (effects (font (size 1.27 1.27)) (justify left))
     )
-    (property "Footprint" "Capacitor_SMD:C_0805_2012Metric" (at 164.7952 40.64 0)
+    (property "Footprint" "Capacitor_SMD:C_0603_1608Metric" (at 164.7952 40.64 0)
       (effects (font (size 1.27 1.27)) hide)
     )
@@
       (effects (font (size 1.27 1.27)) (justify left))
     )
-    (property "Footprint" "Capacitor_SMD:C_0805_2012Metric" (at 174.9552 40.64 0)
+    (property "Footprint" "Capacitor_SMD:C_0603_1608Metric" (at 174.9552 40.64 0)
       (effects (font (size 1.27 1.27)) hide)
     )
@@
       (effects (font (size 1.27 1.27)) (justify left))
     )
-    (property "Footprint" "Capacitor_SMD:C_0805_2012Metric" (at 141.9352 40.64 0)
+    (property "Footprint" "Capacitor_SMD:C_0603_1608Metric" (at 141.9352 40.64 0)
       (effects (font (size 1.27 1.27)) hide)
     )
@@
       (effects (font (size 1.27 1.27)) (justify left))
     )
-    (property "Footprint" "Capacitor_SMD:C_0805_2012Metric" (at 134.3152 40.64 0)
+    (property "Footprint" "Capacitor_SMD:C_0603_1608Metric" (at 134.3152 40.64 0)
       (effects (font (size 1.27 1.27)) hide)
     )
@@
       (effects (font (size 1.27 1.27)) (justify left))
     )
-    (property "Footprint" "Capacitor_SMD:C_1206_3216Metric" (at 70.8152 59.69 0)
+    (property "Footprint" "Capacitor_SMD:C_0603_1608Metric" (at 70.8152 59.69 0)
       (effects (font (size 1.27 1.27)) hide)
     )
@@
       (effects (font (size 1.27 1.27)) (justify left))
     )
-    (property "Footprint" "Capacitor_SMD:C_0805_2012Metric" (at 135.5852 62.23 0)
+    (property "Footprint" "Capacitor_SMD:C_0603_1608Metric" (at 135.5852 62.23 0)
       (effects (font (size 1.27 1.27)) hide)
     )
@@
       (effects (font (size 1.27 1.27)) (justify left))
     )
-    (property "Footprint" "Capacitor_SMD:C_1206_3216Metric" (at 87.3252 59.69 0)
+    (property "Footprint" "Capacitor_SMD:C_0603_1608Metric" (at 87.3252 59.69 0)
       (effects (font (size 1.27 1.27)) hide)
     )
@@
       (effects (font (size 1.27 1.27)) (justify left))
     )
-    (property "Footprint" "Capacitor_SMD:C_0805_2012Metric" (at 263.8552 36.83 0)
+    (property "Footprint" "Capacitor_SMD:C_0603_1608Metric" (at 263.8552 36.83 0)
       (effects (font (size 1.27 1.27)) hide)
     )
@@
       (effects (font (size 1.27 1.27)) (justify left))
     )
-    (property "Footprint" "Capacitor_SMD:C_0805_2012Metric" (at 101.2952 86.36 0)
+    (property "Footprint" "Capacitor_SMD:C_0603_1608Metric" (at 101.2952 86.36 0)
       (effects (font (size 1.27 1.27)) hide)
     )
@@
       (effects (font (size 1.27 1.27)) (justify left))
     )
-    (property "Footprint" "Capacitor_SMD:C_0805_2012Metric" (at 94.9452 86.36 0)
+    (property "Footprint" "Capacitor_SMD:C_0603_1608Metric" (at 94.9452 86.36 0)
       (effects (font (size 1.27 1.27)) hide)
     )
@@
       (effects (font (size 1.27 1.27)) (justify left))
     )
-    (property "Footprint" "Capacitor_SMD:C_0805_2012Metric" (at 337.5152 36.83 0)
+    (property "Footprint" "Capacitor_SMD:C_0603_1608Metric" (at 337.5152 36.83 0)
       (effects (font (size 1.27 1.27)) hide)
     )
@@
       (effects (font (size 1.27 1.27)) (justify left))
     )
-    (property "Footprint" "Capacitor_SMD:C_0805_2012Metric" (at 127.9652 62.23 0)
+    (property "Footprint" "Capacitor_SMD:C_0603_1608Metric" (at 127.9652 62.23 0)
       (effects (font (size 1.27 1.27)) hide)
     )
@@
       (effects (font (size 1.27 1.27)) (justify left))
     )
-    (property "Footprint" "Capacitor_SMD:C_0805_2012Metric" (at 337.5152 85.09 0)
+    (property "Footprint" "Capacitor_SMD:C_0603_1608Metric" (at 337.5152 85.09 0)
       (effects (font (size 1.27 1.27)) hide)
     )
@@
       (effects (font (size 1.27 1.27)) (justify left))
     )
-    (property "Footprint" "Capacitor_SMD:C_0805_2012Metric" (at 75.8952 177.8 0)
+    (property "Footprint" "Capacitor_SMD:C_0603_1608Metric" (at 75.8952 177.8 0)
       (effects (font (size 1.27 1.27)) hide)
     )
@@
       (effects (font (size 1.27 1.27)) (justify left))
     )
-    (property "Footprint" "Capacitor_SMD:C_0805_2012Metric" (at 68.2752 86.36 0)
+    (property "Footprint" "Capacitor_SMD:C_0603_1608Metric" (at 68.2752 86.36 0)
       (effects (font (size 1.27 1.27)) hide)
     )
@@
       (effects (font (size 1.27 1.27)) (justify left))
     )
-    (property "Footprint" "Capacitor_SMD:C_0805_2012Metric" (at 149.5552 40.64 0)
+    (property "Footprint" "Capacitor_SMD:C_0603_1608Metric" (at 149.5552 40.64 0)
       (effects (font (size 1.27 1.27)) hide)
     )
@@
       (effects (font (size 1.27 1.27)) (justify left))
     )
-    (property "Footprint" "Capacitor_SMD:C_0805_2012Metric" (at 182.5752 40.64 0)
+    (property "Footprint" "Capacitor_SMD:C_0603_1608Metric" (at 182.5752 40.64 0)
       (effects (font (size 1.27 1.27)) hide)
     )
@@
       (effects (font (size 1.27 1.27)) (justify left))
     )
-    (property "Footprint" "Capacitor_SMD:C_0805_2012Metric" (at 246.0752 36.83 0)
+    (property "Footprint" "Capacitor_SMD:C_0603_1608Metric" (at 246.0752 36.83 0)
       (effects (font (size 1.27 1.27)) hide)
     )
@@
       (effects (font (size 1.27 1.27)) (justify left))
     )
-    (property "Footprint" "Capacitor_SMD:C_0805_2012Metric" (at 337.5152 134.62 0)
+    (property "Footprint" "Capacitor_SMD:C_0603_1608Metric" (at 337.5152 134.62 0)
       (effects (font (size 1.27 1.27)) hide)
     )
@@
       (effects (font (size 1.27 1.27)) (justify left))
     )
-    (property "Footprint" "Capacitor_SMD:C_0805_2012Metric" (at 107.6452 86.36 0)
-      (effects (font (size 1.27 1.27)) hide)
-    )
+    (property "Footprint" "Capacitor_SMD:C_0603_1608Metric" (at 107.6452 86.36 0)
+      (effects (font (size 1.27 1.27)) hide)
+    )

Commit message: placement amélioré
Parts:
- J11: value ENC1 -> ENCA
- J4: value ENC2 -> ENCB
- J5: value ENC3 -> ENCC
Connections:
- net DIR1: now also U1.38 (PC6); no longer U1.34 (PB12)
- net DIR2: now also U1.34 (PB12); no longer U1.33 (PB11)
- net DIR3: now also U1.33 (PB11); no longer U1.38 (PC6)
- net PWM1: now also U1.37 (PB15); no longer U1.35 (PB13)
- net PWM3: now also U1.35 (PB13); no longer U1.37 (PB15)
Other:
- note added: "Error flag depuis le 1 plutot ?"
Changed lines of the file:
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@@
     (effects (font (size 1.27 1.27)) (justify left bottom))
   )
+  (text "Error flag depuis le 1 plutot ? \n" (at 264.16 165.1 0)
+    (effects (font (size 2 2)) (justify left bottom))
+  )
   (text "Encodeurs Moteurs" (at 222.25 81.28 0)
     (effects (font (size 1.27 1.27)) (justify left bottom))
@@
     )
   )
-  (global_label "DIR3" (shape input) (at 148.59 92.71 180) (fields_autoplaced)
-    (effects (font (size 1.27 1.27)) (justify right))
-    (property "Intersheetrefs" "${INTERSHEET_REFS}" (at 141.2505 92.71 0)
-      (effects (font (size 1.27 1.27)) (justify right) hide)
+  (global_label "DIR3" (shape input) (at 184.15 125.73 0) (fields_autoplaced)
+    (effects (font (size 1.27 1.27)) (justify left))
+    (property "Intersheetrefs" "${INTERSHEET_REFS}" (at 191.4895 125.73 0)
+      (effects (font (size 1.27 1.27)) (justify left) hide)
     )
   )
@@
     )
   )
-  (global_label "DIR1" (shape input) (at 184.15 128.27 0) (fields_autoplaced)
-    (effects (font (size 1.27 1.27)) (justify left))
-    (property "Intersheetrefs" "${INTERSHEET_REFS}" (at 191.4895 128.27 0)
-      (effects (font (size 1.27 1.27)) (justify left) hide)
+  (global_label "DIR1" (shape input) (at 148.59 92.71 180) (fields_autoplaced)
+    (effects (font (size 1.27 1.27)) (justify right))
+    (property "Intersheetrefs" "${INTERSHEET_REFS}" (at 141.2505 92.71 0)
+      (effects (font (size 1.27 1.27)) (justify right) hide)
     )
   )
@@
     )
   )
-  (global_label "PWM3" (shape input) (at 184.15 135.89 0) (fields_autoplaced)
+  (global_label "PWM3" (shape input) (at 184.15 130.81 0) (fields_autoplaced)
     (effects (font (size 1.27 1.27)) (justify left))
-    (property "Intersheetrefs" "${INTERSHEET_REFS}" (at 192.5175 135.89 0)
+    (property "Intersheetrefs" "${INTERSHEET_REFS}" (at 192.5175 130.81 0)
       (effects (font (size 1.27 1.27)) (justify left) hide)
     )
@@
     )
   )
-  (global_label "PWM1" (shape input) (at 184.15 130.81 0) (fields_autoplaced)
+  (global_label "PWM1" (shape input) (at 184.15 135.89 0) (fields_autoplaced)
     (effects (font (size 1.27 1.27)) (justify left))
-    (property "Intersheetrefs" "${INTERSHEET_REFS}" (at 192.5175 130.81 0)
+    (property "Intersheetrefs" "${INTERSHEET_REFS}" (at 192.5175 135.89 0)
       (effects (font (size 1.27 1.27)) (justify left) hide)
     )
@@
     )
   )
-  (global_label "DIR2" (shape input) (at 184.15 125.73 0) (fields_autoplaced)
+  (global_label "DIR2" (shape input) (at 184.15 128.27 0) (fields_autoplaced)
     (effects (font (size 1.27 1.27)) (justify left))
-    (property "Intersheetrefs" "${INTERSHEET_REFS}" (at 191.4895 125.73 0)
+    (property "Intersheetrefs" "${INTERSHEET_REFS}" (at 191.4895 128.27 0)
       (effects (font (size 1.27 1.27)) (justify left) hide)
     )
@@
       (effects (font (size 1.27 1.27)))
     )
-    (property "Value" "ENC3" (at 274.955 87.63 0)
+    (property "Value" "ENCC" (at 274.955 87.63 0)
       (effects (font (size 1.27 1.27)))
     )
@@
       (effects (font (size 1.27 1.27)))
     )
-    (property "Value" "ENC2" (at 255.905 87.63 0)
+    (property "Value" "ENCB" (at 255.905 87.63 0)
       (effects (font (size 1.27 1.27)))
     )
@@
       (effects (font (size 1.27 1.27)))
     )
-    (property "Value" "ENC1" (at 235.585 87.63 0)
+    (property "Value" "ENCA" (at 235.585 87.63 0)
       (effects (font (size 1.27 1.27)))
     )
