File: Brushless/CarteBrushless.kicad_pcb (KiCad board)
At the start: 2 copper layers, 68 x 84 mm, 71 parts, among them Q2 IRF7424, U1 STM32G484RETx

Commit message: placement PCB
Parts:
- removed C1, C3, C5: 100n, Capacitor_SMD:C_0603_1608Metric
- removed C2, C4, C6: 100u, Capacitor_SMD:CP_Elec_10x12.5
- removed ENC 1: ENC1, Connector_PinHeader_2.54mm:PinHeader_1x04_P2.54mm_Vertical
- removed ENC 2: ENC2, Connector_PinHeader_2.54mm:PinHeader_1x04_P2.54mm_Vertical
- removed ENC 3: ENC3, Connector_PinHeader_2.54mm:PinHeader_1x04_P2.54mm_Vertical
- removed the G*** at (121.0, 100.0)
- removed U3, U6: ~, ENAC_robotique:IFX9201SG
- removed locked: MOT3, TerminalBlock:TerminalBlock_bornier-2_P5.08mm
- removed locked: MOT2, TerminalBlock:TerminalBlock_bornier-2_P5.08mm
- removed locked: MOT1, TerminalBlock:TerminalBlock_bornier-2_P5.08mm
- added D1: D, Diode_SMD:Nexperia_CFP3_SOD-123W, F.Cu at (126.5, 131.4)
- added J1: Conn_01x03_Pin, Connector_Molex:Molex_PicoBlade_53398-0371_1x03-1MP_P1.25mm_Vertical, F.Cu at (136.5, 94.6)
- added J2: Conn_01x03_Pin, Connector_Molex:Molex_PicoBlade_53398-0371_1x03-1MP_P1.25mm_Vertical, F.Cu at (136.5, 109.8)
- added J3: Conn_01x03_Pin, Connector_Molex:Molex_PicoBlade_53398-0371_1x03-1MP_P1.25mm_Vertical, F.Cu at (136.5, 124.4)
- added JP1: SolderJumper_2_Open, Jumper:SolderJumper-2_P1.3mm_Open_RoundedPad1.0x1.5mm, F.Cu at (128.3, 121.9)
- added JP2: SolderJumper_2_Open, Jumper:SolderJumper-2_P1.3mm_Open_RoundedPad1.0x1.5mm, F.Cu at (139.7, 88.9)
- added MOT1: MOT3, Connector_AMASS:AMASS_XT30UPB-F_1x02_P5.0mm_Vertical, F.Cu at (150.5, 92.7)
- added MOT2: MOT3, Connector_AMASS:AMASS_XT30UPB-F_1x02_P5.0mm_Vertical, F.Cu at (150.5, 107.3)
- added MOT3: MOT3, Connector_AMASS:AMASS_XT30UPB-F_1x02_P5.0mm_Vertical, F.Cu at (150.5, 121.9)
- added R11: 120, Resistor_SMD:R_0805_2012Metric, F.Cu at (135.3, 89.2)
- C23: value 10u -> 100u; footprint Capacitor_SMD:C_0603_1608Metric -> Capacitor_Tantalum_SMD:CP_EIA-7343-31_Kemet-D_Pad2.25x2.55mm_HandSolder
- R1: value 10k -> 120
- TP_CS1, TP_GND1, TP_MISO1, TP_MOSI1, TP_SCK1: footprint TestPoint:TestPoint_Pad_D2.0mm -> TestPoint:TestPoint_Pad_D1.5mm
- U2: value ~ -> TCAN332G; footprint ENAC_robotique:IFX9201SG -> Package_TO_SOT_SMD:SOT-23-8
- UART1: renamed from UART4; footprint Connector_PinHeader_2.54mm:PinHeader_1x03_P2.54mm_Vertical -> Connector_Molex:Molex_PicoBlade_53398-0371_1x03-1MP_P1.25mm_Vertical
- moved UART1 41.5 mm to (101.8, 119.4), turned to -90 degrees
- moved LED2 37.0 mm to (102.5, 113.0), turned to 0 degrees
- moved LED1 34.7 mm to (102.5, 106.7), turned to 0 degrees
- moved R10 33.8 mm to (102.5, 108.7), turned to 180 degrees
- moved R6 33.1 mm to (102.5, 111.0), turned to 180 degrees
- moved G*** 31.6 mm to (69.2, 82.5)
- moved SWITCH1 26.3 mm to (111.7, 86.6), turned to 180 degrees
- moved R9 25.0 mm to (112.1, 89.8), turned to 0 degrees
- moved R4 20.5 mm to (109.9, 124.2)
- moved DEBUG1 19.9 mm to (125.0, 100.3)
- moved R7 19.5 mm to (126.7, 92.1)
- moved R8 19.5 mm to (121.9, 92.1)
- moved USB-C1 19.5 mm to (124.5, 84.5)
- moved U2 18.4 mm to (127.6, 115.9), turned to 0 degrees
- moved D3 17.3 mm to (117.9, 89.4), turned to -90 degrees
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Connections:
- C23 pad 1: +BATT -> Net-(D1-K)
- R1 pad 1: +3.3V -> Net-(JP1-B)
- R1 pad 2: DIS -> CAN_HIGH
- Transfo18->5 pad 1: +BATT -> Net-(D1-K)
- U1 pad 10: unconnected-(U1-PC2-Pad10) -> LED2
- U1 pad 12: Enc2_B -> unconnected-(U1-PA0-Pad12)
- U1 pad 13: Enc2_A -> unconnected-(U1-PA1-Pad13)
- U1 pad 14: unconnected-(U1-PA2-Pad14) -> UART2_TX
- U1 pad 17: unconnected-(U1-PA3-Pad17) -> UART2_RX
- U1 pad 18: unconnected-(U1-PA4-Pad18) -> MEAS_VBAT
- U1 pad 20: Enc1_A -> unconnected-(U1-PA6-Pad20)
- U1 pad 21: Enc1_B -> unconnected-(U1-PA7-Pad21)
- U1 pad 33: DIR2 -> unconnected-(U1-PB11-Pad33)
- U1 pad 34: DIR3 -> CAN_RX
- U1 pad 35: PWM3 -> CAN_TX
- U1 pad 36: PWM2 -> unconnected-(U1-PB14-Pad36)
- U1 pad 37: PWM1 -> unconnected-(U1-PB15-Pad37)
- U1 pad 38: DIR1 -> unconnected-(U1-PC6-Pad38)
- U1 pad 39: DIS -> unconnected-(U1-PC7-Pad39)
- U1 pad 40: ERROR_FLAG -> unconnected-(U1-PC8-Pad40)
- U1 pad 42: MEAS_VBAT -> unconnected-(U1-PA8-Pad42)
- U1 pad 43: LED1 -> unconnected-(U1-PA9-Pad43)
- U1 pad 44: LED2 -> unconnected-(U1-PA10-Pad44)
- U1 pad 52: UART4_TX -> unconnected-(U1-PC10-Pad52)
- U1 pad 53: UART4_RX -> unconnected-(U1-PC11-Pad53)
- U1 pad 54: IMU_INT1 -> unconnected-(U1-PC12-Pad54)
- U1 pad 55: SPI1_CS_IMU -> IMU_INT1
- U1 pad 59: Enc3_B -> SPI1_CS_IMU
- U1 pad 60: Enc3_A -> unconnected-(U1-PB7-Pad60)
- U1 pad 9: unconnected-(U1-PC1-Pad9) -> LED1
- U2 pad 1: DIR2 -> CAN_TX
- U2 pad 2: +3.3V -> GND
- U2 pad 3: Net-(U2-SO) -> +3.3V
- U2 pad 4: +BATT -> CAN_RX
- U2 pad 5: Net-(MOT2-Pin_1) -> unconnected-(U2-NC-Pad5)
- U2 pad 6: GND -> CAN_LOW
- U2 pad 7: Net-(MOT2-Pin_2) -> CAN_HIGH
- U2 pad 8: Net-(U2-SI) -> unconnected-(U2-NC-Pad8)
- UART1 pad 2: UART4_TX -> UART2_TX
- UART1 pad 3: UART4_RX -> UART2_RX
Routing:
- net +3.3V: track 196.4 -> 0.00 mm, vias 10 -> 0
- net GND: track 201.7 -> 8.91 mm, vias 70 -> 0
- net +5V: track 132.1 -> 35.1 mm
- net DIS: track 84.5 -> 0.00 mm, vias 6 -> 0
- net PWM1: track 51.7 -> 0.00 mm, vias 2 -> 0
- net USB_DP: track 48.7 -> 0.00 mm
- net USB_DM: track 48.6 -> 0.00 mm
- net DIR1: track 41.2 -> 0.00 mm
- net RST: track 41.0 -> 0.00 mm
- net UART4_TX: track 30.9 -> 0.00 mm
- net ERROR_FLAG: track 28.7 -> 0.00 mm, vias 2 -> 0
- net UART4_RX: track 28.1 -> 0.00 mm
- net SWCLK: track 27.9 -> 0.00 mm
- net PWM2: track 27.8 -> 0.00 mm
- net LED1: track 27.1 -> 0.00 mm
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- removed copper zone on B.Cu, net +BATT
- removed copper zone on F.Cu, net +BATT
- removed copper zone on B.Cu, net GND
- removed copper zone on F.Cu, net Net-(MOT1-Pin_1)
- removed copper zone on F.Cu, net Net-(MOT1-Pin_2)
- removed copper zone on F.Cu, net Net-(MOT2-Pin_1)
- removed copper zone on F.Cu, net Net-(MOT2-Pin_2)
- removed copper zone on F.Cu, net Net-(MOT3-Pin_1)
- removed copper zone on F.Cu, net Net-(MOT3-Pin_2)
Other:
- board text added: "SWD"
- board text removed: "A"
- board text removed: "B"
- board text removed: "LED"
- board text removed: "SW"

Commit message: Routage fini
Parts:
- added G***: LOGO, ENAC_robotique:logo_enac_mini, F.Cu at (144.5, 138.7)
- G***: moved to B.Cu
- moved G*** 64.7 mm to (132.0, 98.3), turned to 180 degrees
- moved H1 21.2 mm to (100.0, 86.2)
- moved H2 19.2 mm to (152.0, 86.2)
- moved H4 9.04 mm to (100.0, 142.2)
- moved ALIM1 6.11 mm to (114.9, 140.5)
- moved Q2 6.11 mm to (120.7, 131.6)
- moved C19 6.11 mm to (112.4, 134.4)
- moved D5 6.11 mm to (113.9, 130.7)
- moved R2 6.11 mm to (116.2, 130.7)
- moved R5 6.11 mm to (111.6, 130.1)
- moved Transfo5->3.3 6.11 mm to (107.4, 136.2)
- moved C23 5.69 mm to (126.9, 135.0)
- moved C24 5.69 mm to (125.5, 141.7)
- moved D2 5.69 mm to (128.5, 142.0)
- moved C21 5.68 mm to (106.7, 128.8)
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Connections:
- DEBUG1 pad 1: GND -> SWDIO
- DEBUG1 pad 2: +3.3V -> SWCLK
- DEBUG1 pad 4: SWCLK -> +3.3V
- DEBUG1 pad 5: SWDIO -> GND
- UART1 pad 2: UART2_TX -> UART2_RX
- UART1 pad 3: UART2_RX -> UART2_TX
Routing:
- net +3.3V: track 0.00 -> 136.7 mm, vias 0 -> 4
- net GND: track 8.91 -> 138.1 mm, vias 0 -> 16
- net CAN_LOW: track 0.00 -> 49.3 mm
- net CAN_HIGH: track 0.00 -> 47.9 mm, vias 0 -> 3
- net +5V: track 35.1 -> 75.1 mm, vias 0 -> 3
- net USB_DM: track 0.00 -> 30.0 mm
- net USB_DP: track 0.00 -> 28.2 mm
- net RST: track 0.00 -> 23.8 mm
- net /BOOT 0: track 0.00 -> 23.2 mm
- net SPI1_MOSI: track 0.00 -> 16.2 mm, vias 0 -> 2
- net SPI1_SCK: track 0.00 -> 16.2 mm, vias 0 -> 3
- net SPI1_CS_IMU: track 0.00 -> 15.3 mm, vias 0 -> 2
- net UART2_RX: track 0.00 -> 14.9 mm
- net SPI1_MISO: track 0.00 -> 14.4 mm, vias 0 -> 2
- net VBUS: track 0.00 -> 14.3 mm, vias 0 -> 3
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- added copper zone on F.Cu, net +BATT
- added copper zone on B.Cu, net GND
Other:
- board size 68 x 84 mm -> 60 x 64 mm
- board text added: "Base Roulante Brushless V1 Edition 2025 by Hugo@Enac"
- board text added: "Base Roulante Brushless V1 by Hugo@Enac"
- board text removed: "Base Roulante 2024 by Hugo@Enac"
